Commit message: Updated URDFReader with bugfixes; convex contact reduction now checks for equal coefficients of friction

File: example/HyQ/hyq.urdf (robot description, URDF)
Before this commit: robot hyq, 17 links, 16 joints
Links:
- link LF_HIP_FE: mass 2.482000 -> 1.772; geometry collision mesh filename=ycyl-r0.01-l0.35.obj; visual mesh filename=ycyl-r0.01-l0.35.obj
- link LF_KNEE: geometry collision mesh filename=ycyl-r0.01-l0.33.obj; visual mesh filename=ycyl-r0.01-l0.33.obj
Joints:
- joint LF_HAA: origin xyz=0.3735 0.207 0.0 rpy=3.141593 1.570796 0.0 -> xyz=0.3735 0.207 0.0 rpy=0 -1.570796 -3.141593
- joint LF_LLF: origin xyz=0.33 0.0 0.0 rpy=0.0 -1.570796 -1.570796 -> xyz=0.33 0.0 0.0 rpy=0.0 0.0 0.0

Commit message: Bugfix to ATLAS bug; URDFReader now works properly

File: example/HyQ/hyq.urdf (robot description, URDF)
Before this commit: robot hyq, 17 links, 16 joints
Links:
- link LH_HIP_FE: geometry collision mesh filename=ycyl-r0.01-l0.35.obj; visual mesh filename=ycyl-r0.01-l0.35.obj
- link LH_KNEE: geometry collision mesh filename=ycyl-r0.01-l0.33.obj; visual mesh filename=ycyl-r0.01-l0.33.obj
- link RF_HIP_FE: geometry collision mesh filename=ycyl-r0.01-l0.35.obj; visual mesh filename=ycyl-r0.01-l0.35.obj
- link RF_KNEE: geometry collision mesh filename=ycyl-r0.01-l0.33.obj; visual mesh filename=ycyl-r0.01-l0.33.obj
- link RH_HIP_FE: geometry collision mesh filename=ycyl-r0.01-l0.35.obj; visual mesh filename=ycyl-r0.01-l0.35.obj
- link RH_KNEE: geometry collision mesh filename=ycyl-r0.01-l0.33.obj; visual mesh filename=ycyl-r0.01-l0.33.obj
Joints:
- joint LF_HAA: origin xyz=0.3735 0.207 0.0 rpy=0 -1.570796 -3.141593 -> xyz=0.3735 0.207 0.0 rpy=0 1.570796 3.141593
- joint RF_HAA: origin xyz=0.3735 -0.207 0.0 rpy=3.141593 1.570796 3.141593 -> xyz=0.3735 -0.207 0.0 rpy=0 1.570796 0

Commit message: Fixed generalized force calculation for CRBAlgorithm

File: example/HyQ/hyq.urdf (robot description, URDF)
Before this commit: robot hyq, 17 links, 16 joints
Links:
- link LF_HIP_FE: geometry collision mesh filename=/home/samzapo/Moby/example/HyQ/ycyl-r0.01-l0.35.obj; visual mesh filename=/home/samzapo/Moby/example/HyQ/ycyl-r0.01-l0.35.obj
- link LF_KNEE: geometry collision mesh filename=/home/samzapo/Moby/example/HyQ/ycyl-r0.01-l0.33.obj; visual mesh filename=/home/samzapo/Moby/example/HyQ/ycyl-r0.01-l0.33.obj
- link LH_HIP_FE: geometry collision mesh filename=/home/samzapo/Moby/example/HyQ/ycyl-r0.01-l0.35.obj; visual mesh filename=/home/samzapo/Moby/example/HyQ/ycyl-r0.01-l0.35.obj
- link LH_KNEE: geometry collision mesh filename=/home/samzapo/Moby/example/HyQ/ycyl-r0.01-l0.33.obj; visual mesh filename=/home/samzapo/Moby/example/HyQ/ycyl-r0.01-l0.33.obj
- link RF_HIP_FE: geometry collision mesh filename=/home/samzapo/Moby/example/HyQ/ycyl-r0.01-l0.35.obj; visual mesh filename=/home/samzapo/Moby/example/HyQ/ycyl-r0.01-l0.35.obj
- link RF_KNEE: geometry collision mesh filename=/home/samzapo/Moby/example/HyQ/ycyl-r0.01-l0.33.obj; visual mesh filename=/home/samzapo/Moby/example/HyQ/ycyl-r0.01-l0.33.obj
- link RH_HIP_FE: geometry collision mesh filename=/home/samzapo/Moby/example/HyQ/ycyl-r0.01-l0.35.obj; visual mesh filename=/home/samzapo/Moby/example/HyQ/ycyl-r0.01-l0.35.obj
- link RH_KNEE: geometry collision mesh filename=/home/samzapo/Moby/example/HyQ/ycyl-r0.01-l0.33.obj; visual mesh filename=/home/samzapo/Moby/example/HyQ/ycyl-r0.01-l0.33.obj

Commit message: Fixed a few bugs in RCArticulatedBody event calculation for floating bases

File: example/HyQ/hyq.urdf (robot description, URDF)
Before this commit: robot hyq, 17 links, 16 joints
Links:
- link LF_FOOT: mass 0.0 -> 0.001
- link LH_FOOT: mass 0.0 -> 0.001
- link RF_FOOT: mass 0.0 -> 0.001
- link RH_FOOT: mass 0.0 -> 0.001
