Commit message: Create compliant layer branch

File: example/urdf/pendulum.urdf (robot description, URDF)
Before this commit: robot pendulum, 3 links, 2 joints
Links:
- removed link pendulum_link
- removed link pendulum_rod_link
- added link pendulum_bob, mass 0.05; collision sphere radius=0.03; visual sphere radius=0.03
- added link pendulum_rod, mass 0.001; collision cylinder length=0.25 radius=0.01; visual cylinder length=0.25 radius=0.01
Joints:
- joint pendulum_fixed_joint: child pendulum_rod_link -> pendulum_rod; parent pendulum_link -> pendulum_bob
- joint pendulum_joint: child pendulum_link -> pendulum_bob; origin xyz=0 0.18 0.0 rpy=0 0 0 -> xyz=0 0 0.0 rpy=0 0 0
